Commit message: add mapping.launch

File: src/my_robot/urdf/my_robot.xacro (robot description, xacro)
@@ -161,4 +161,11 @@
       </geometry>
     </collision>
+  </link>
+  <joint name="camera_optical_joint" type="fixed">
+    <origin xyz="0 0 0" rpy="-1.5707 0 -1.5707"/>
+    <parent link="camera"/>
+    <child link="camera_link_optical"/>
+  </joint>
+  <link name="camera_link_optical">
   </link>
   <!-- Lidar Link -->
